File: K40Optokoppler.kicad_pcb (KiCad board)
At the start: 2 copper layers, 9 parts, among them J1 Conn_01x02_Male, J2 Conn_01x04, U1 TLP627-2

Commit message: Step-Datei
Step-Datei der Platine hinzugefügt
Other:
- board outline added: 41.9 x 30.5 mm
Changed lines of the file:
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@@
   (general
     (thickness 1.6)
-    (drawings 4)
+    (drawings 8)
     (tracks 32)
     (zones 0)
@@
     )
   )
+  (gr_line (start 29.21 87.63) (end 29.21 57.15) (layer Edge.Cuts) (width 0.15))
+  (gr_line (start 71.12 87.63) (end 29.21 87.63) (layer Edge.Cuts) (width 0.15))
+  (gr_line (start 71.12 57.15) (end 71.12 87.63) (layer Edge.Cuts) (width 0.15))
+  (gr_line (start 29.21 57.15) (end 71.12 57.15) (layer Edge.Cuts) (width 0.15))
   (gr_line (start 29.21 87.63) (end 29.21 57.15) (layer F.SilkS) (width 0.2))
   (gr_line (start 71.12 87.63) (end 29.21 87.63) (layer F.SilkS) (width 0.2))
